File: Wireless RIFID Reader PCB/Wireless RIFID Reader.brd (EAGLE design)
At the start: 25.4 x 61.6 mm, 33 parts, among them J1 FCI: 10103594-0001LF, J2 4UCON 20404, J3 Antenna, J4 ICD3, J5 NeoPixels, U1 PIC32MX470F512H-I/PT, U2 MIC5319-3.3YD5, U3 ID-3LA, U4 MCP73832T-2ACI/OT

Commit message: Commit PCB v1.1 files
Parts:
- added C13: 220u, Case D, rcl:SMC_D
- added J11: (no value), SparkFun-Passives:PAD-JUMPER-3-NO_YES_SILK_FULL_BOX
- added LED1: RS: 654-4304, SparkFun:LED-0603
- added Q1: IRLML6401, SparkFun:SOT23
- added Q2, Q3: MMBT2222A, SparkFun-DiscreteSemi:SOT23-3
- added R5: 10k 0603, SparkFun:0402-RES
- added R6, R7, R8: 1k, 0603, SparkFun:0402-RES
- added SG1: BUZZERSMD2, SparkFun-Electromechanical:BUZZER-CCV
- C7: value 4u7, 0603 -> 10u, 0603
- moved LOGO1 20.4 mm to (11.4, 34.9)
- moved J6 3.18 mm to (8.89, 28.6)
- moved J7 3.18 mm to (11.4, 28.6)
- moved J8 3.18 mm to (14.0, 28.6)
- moved J9 3.18 mm to (16.5, 28.6)
- moved U3 0.90 mm to (11.4, 14.6)
Connections:
- net BATT_LEVEL renamed BATTERY_LEVEL
- removed net CHRG_STAT: U4.1
- new net BUZZER: J11.1, U1.63
- new net N$10: Q3.1, R8.1
- new net N$12: Q3.3, SG1.+
- new net N$13: J11.3, U3.10
- new net N$15: J11.2, R8.2
- new net N$4: J5.2, Q1.3
- new net N$5: Q1.1, Q2.3, R5.1
- new net N$6: Q2.1, R6.1
- new net N$9: LED1.A, R7.2
- new net NEOPIXEL_ENABLE: R6.2, U1.1
- new net STAT: U1.29, U4.1
- net GND: now also C13.-, LED1.C, Q2.2, Q3.2
- net VBATT: now also C13.+, Q1.2, R5.2, SG1.-; no longer J5.2
- net VDD: now also R7.1
- net XBEE_DIN: now also U1.51; no longer U1.50
- net XBEE_DOUT: now also U1.48; no longer U1.51
Routing:
- net STAT: track 0.00 -> 38.3 mm, vias 0 -> 2
- net N$4: track 0.00 -> 16.0 mm
- net BUZZER: track 0.00 -> 14.5 mm, vias 0 -> 1
- net N$12: track 0.00 -> 12.3 mm
- net N$13: track 0.00 -> 8.85 mm
- net N$5: track 0.00 -> 5.43 mm
- net N$15: track 0.00 -> 4.58 mm
- net NEOPIXEL_ENABLE: track 0.00 -> 4.34 mm, vias 0 -> 1
- net N$9: track 0.00 -> 4.27 mm
- net SEL0: track 9.04 -> 5.15 mm
- net SEL1: track 9.81 -> 6.63 mm
- net N$10: track 0.00 -> 2.84 mm
- net SEL2: track 9.27 -> 6.45 mm
- net XBEE_DOUT: track 16.9 -> 14.1 mm
- net N$6: track 0.00 -> 2.30 mm
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Other:
- board text added: "DOUT"
- board text added: "POWER"
- board text added: "Wireless RFID Reader v1.1"
- board text removed: "BATTERY"
- board text removed: "NEOPIXEL DATA"
- board text removed: "Wireless RFID Reader"
