File: Wireless RIFID Reader PCB/Wireless RIFID Reader.sch (EAGLE design)
At the start: 33 parts, among them J1 FCI: 10103594-0001LF, J2 4UCON 20404, J3 Antenna, J4 ICD3, J5 NeoPixels, U1 PIC32MX470F512H-I/PT, U2 MIC5319-3.3YD5, U3 ID-3LA, U4 MCP73832T-2ACI/OT

Commit message: Commit PCB v1.1 files
Parts:
- added C13: 220u, Case D, rcl:CPOL-USSMCD
- added J11: JUMPER-PAD-3-NOFULL_BOX_SILK, SparkFun-Passives:JUMPER-PAD-3-NOFULL_BOX_SILK
- added LED1: RS: 654-4304, SparkFun:LED0603
- added Q1: IRLML6401, SparkFun:MOSFET-PCHANNEL
- added Q2, Q3: MMBT2222A, SparkFun-DiscreteSemi:TRANSISTOR_NPNMMBT2222A
- added R5: 10k 0603, SparkFun:RESISTOR0402-RES
- added R6, R7, R8: 1k, 0603, SparkFun:RESISTOR0402-RES
- added SG1: BUZZERSMD2, SparkFun-Electromechanical:BUZZERSMD2
- C7: value 4u7, 0603 -> 10u, 0603
- S1: device x-io:SWITCH-DPST -> x-io:SWITCH-DPSTMMP122-R
Connections:
- net BATT_LEVEL renamed BATTERY_LEVEL
- removed net CHRG_STAT: U4.STAT
- new net BUZZER: J11.1, U1.TRD3/RPE3/CTPLS/PMD3/RE3
- new net N$10: Q3.B, R8.1
- new net N$12: Q3.C, SG1.1
- new net N$13: J11.3, U3.READ
- new net N$15: J11.2, R8.2
- new net N$4: J5.2, Q1.D
- new net N$5: Q1.G, Q2.C, R5.1
- new net N$6: Q2.B, R6.1
- new net N$9: LED1.A, R7.2
- new net NEOPIXEL_ENABLE: R6.2, U1.AN22/RPE5/PMD5/RE5
- new net STAT: U1.AN14/RPB14/CTED5/PMA1/RB14, U4.STAT
- net GND: now also C13.-, LED1.C, Q2.E, Q3.E
- net VBATT: now also C13.+, Q1.S, R5.2, SG1.2; no longer J5.2
- net VDD: now also R7.1
- net XBEE_DIN: now also U1.AN26/RPD3/RD3; no longer U1.AN25/RPD2/SCK1/RD2
- net XBEE_DOUT: now also U1.SOSCO/RPC14/T1CK/RC14; no longer U1.AN26/RPD3/RD3
Other:
- note added: "Power LED"
- moved on the sheet: C1, C10, C11, C2, C3, C4, C5, C6, C7, C8, C9, J1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
